File: PCB/Spikeling_V2.2c.kicad_pcb (KiCad board)
At the start: 2 copper layers, 120 x 80 mm, 52 parts, among them J1 Synapse Out, J2 Synapse in 1, J4 Current in, J5 Stimulus Out, SW1 Mode Button, SW2 Reset Button, U1 ESP32-DEVKITC-32D, U2 MCP3208, U3 MCP3208

Commit message: update PCB
Parts:
- removed the D1 at (140.0, 124.4)
- added R10: R_Photo, Maxime:Photoresistor_3.4, F.Cu at (138.3, 124.4)
- added R11: 10kΩ, Resistor_THT:R_Axial_DIN0207_L6.3mm_D2.5mm_P10.16mm_Horizontal, F.Cu at (176.6, 111.6)
- added SW2: Buzzer Button, Button_Switch_THT:Spikeling reset button, F.Cu at (195.0, 50.1)
- C3: footprint Capacitor_THT:C_Disc_D10.0mm_W2.5mm_P5.00mm -> Capacitor_THT:CP_Radial_D4.0mm_P2.00mm
- U1: footprint Module:MODULE_ESP32-DEVKITC-32D -> Maxime:MODULE_ESP32-DEVKITC-32D
- moved kibuzzard-633362FE 64.0 mm to (159.8, 110.0)
- moved SW3 4.56 mm to (130.0, 50.1)
- renumbered D14 to D1, e to J3, SW2 to SW3
Connections:
- D1 pad 1: /27 -> Net-(D1-Pad2)
- D1 pad 2: Net-(R4-Pad2) -> /27
- R4 pad 2: Net-(R4-Pad2) -> Net-(D1-Pad2)
- U1 pad 3: unconnected-(U1-Pad3) -> /36
Routing:
- net /36: track 0.00 -> 78.3 mm
- net VCC: track 345.5 -> 388.6 mm
- net Net-(SW3-Pad2): track 92.8 -> 127.9 mm, vias 1 -> 0
- net Net-(D1-Pad2): track 0.00 -> 21.1 mm
- net Net-(R4-Pad2): track 13.4 -> 0.00 mm
- net /106: track 72.4 -> 76.4 mm, vias 0 -> 1
- net Net-(C3-Pad1): track 13.7 -> 16.2 mm
- net /100: track 65.4 -> 67.4 mm
- net /15: track 71.5 -> 70.5 mm
- net /27: track 48.3 -> 49.1 mm
- net Net-(D10-Pad2): track 50.6 -> 49.8 mm
- net GNDREF: track 0.72 -> 0.00 mm
Other:
- board text added: "Spike button Resistor"
- board text removed: "An Open Source Hardware implementation of a spiking neuron for neuroscience teaching and outreach"
- board text removed: "Spikeling v2.2"
