File: PCB/Spikeling_V2.2c.kicad_sch (KiCad schematic)
At the start: 44 parts, among them U1 ESP32-DEVKITC-32D, U2 MCP3208, U3 MCP3208

Commit message: update PCB
Parts:
- removed D1: (no value), symbol Device:D_Photo
- added R10: (no value), symbol Device:R_Photo
- added R11: (no value), symbol Device:R
- added SW2: (no value), symbol Switch:SW_Push
- BZ1: value (none) -> Spike Buzzer; footprint (none) -> Buzzer_Beeper:Buzzer_11.5x9.5RM5
- C1: value (none) -> 1 μF; footprint (none) -> Capacitor_THT:CP_Radial_D4.0mm_P2.00mm
- C3: value (none) -> 1nF; footprint (none) -> Capacitor_THT:CP_Radial_D4.0mm_P2.00mm
- D1: renamed from D14; value (none) -> Spike LED; footprint (none) -> LED_THT:LED_D5.0mm-4_RGB
- D10: value (none) -> Mode9; footprint (none) -> LED_THT:LED_D3.0mm
- D11: value (none) -> Mode10; footprint (none) -> LED_THT:LED_D3.0mm
- D12: value (none) -> Mode11; footprint (none) -> LED_THT:LED_D3.0mm
- D13: value (none) -> Mode12; footprint (none) -> LED_THT:LED_D3.0mm
- D2: value (none) -> Mode1; footprint (none) -> LED_THT:LED_D3.0mm
- D3: value (none) -> Mode2; footprint (none) -> LED_THT:LED_D3.0mm
- D4: value (none) -> Mode3; footprint (none) -> LED_THT:LED_D3.0mm
- D5: value (none) -> Mode4; footprint (none) -> LED_THT:LED_D3.0mm
- D6: value (none) -> Mode5; footprint (none) -> LED_THT:LED_D3.0mm
- D7: value (none) -> Mode6; footprint (none) -> LED_THT:LED_D3.0mm
- D8: value (none) -> Mode7; footprint (none) -> LED_THT:LED_D3.0mm
- D9: value (none) -> Mode8; footprint (none) -> LED_THT:LED_D3.0mm
- J1: value (none) -> Synapse Out; footprint (none) -> Audio_Module:Spikeling Audio Jack 3.5mm
- J2: value (none) -> Synapse in 1; footprint (none) -> Audio_Module:Spikeling Audio Jack 3.5mm
- J3: value (none) -> Synapse in 2; footprint (none) -> Audio_Module:Spikeling Audio Jack 3.5mm
- J4: value (none) -> Current in; footprint (none) -> Audio_Module:Spikeling Audio Jack 3.5mm
- J5: value (none) -> Stimulus Out; footprint (none) -> Audio_Module:Spikeling Audio Jack 3.5mm
- R1: value (none) -> 10Ω; footprint (none) -> Resistor_THT:R_Axial_DIN0207_L6.3mm_D2.5mm_P10.16mm_Horizontal
- R2, R5: value (none) -> 10kΩ; footprint (none) -> Resistor_THT:R_Axial_DIN0207_L6.3mm_D2.5mm_P10.16mm_Horizontal
- R3, R4, R6, R7, R8, R9: value (none) -> 100Ω; footprint (none) -> Resistor_THT:R_Axial_DIN0207_L6.3mm_D2.5mm_P10.16mm_Horizontal
- RV1: value (none) -> Synapse 1 Gain; footprint (none) -> Potentiometer_THT:Spikeling Potentiometer
- RV2: value (none) -> Synapse 2 Gain; footprint (none) -> Potentiometer_THT:Spikeling Potentiometer
- RV3: value (none) -> Voltage Membrane; footprint (none) -> Potentiometer_THT:Spikeling Potentiometer
- RV4: value (none) -> Noise; footprint (none) -> Potentiometer_THT:Spikeling Potentiometer
- RV5: value (none) -> Photodiode Gain; footprint (none) -> Potentiometer_THT:Spikeling Potentiometer
- RV6: value (none) -> Stimulus Strength; footprint (none) -> Potentiometer_THT:Spikeling Potentiometer
- RV7: value (none) -> Stimulus Frequency; footprint (none) -> Potentiometer_THT:Spikeling Potentiometer
- SW1: value (none) -> Mode Button; footprint (none) -> Button_Switch_THT:SW_PUSH_6mm_H13mm
- SW3: renamed from SW2; value (none) -> Reset Button; footprint (none) -> Button_Switch_THT:Spikeling reset button
Connections:
- net 202: now also R10.1
- net GNDREF: now also R11.2
- net VCC: now also R10.2, SW2.2
- net 36: now reaches U1.3 (SENSOR_VP)
- net 36: now also R11.1, SW2.1
- no-connect marks 10 -> 9
Other:
- moved on the sheet: C3, J1, J5, R1, R3, R5, RV6, RV7, SW1
